File: plate/plate6_dx/plate6_dx.kicad_pcb (KiCad board)
At the start: 2 copper layers, 163.6 x 113.2 mm, 0 parts

Commit message: tastiera con rj11 mandata in stampa
Other:
- outline, holes or cut-outs redrawn
